File: hw1/hw1.kicad_pcb (KiCad board)
At the start: 2 copper layers, 68.6 x 53.3 mm, 8 parts, among them P1 Power, P2 Analog, P3 Digital, P4 Digital, P5 CONN_01X01, P6 CONN_01X01, P7 CONN_01X01, P8 CONN_01X01

Commit message: hw1: schematic "finished" ?
have I committed enough files for others to even open this?
Parts:
- added C1: 100n, Capacitors_SMD:C_0603_HandSoldering, F.Cu at (144.4, 100.1)
- added C2: 100n, Capacitors_SMD:C_0603_HandSoldering, F.Cu at (157.0, 108.7)
- added C3: 100n, Capacitors_SMD:C_0603_HandSoldering, F.Cu at (144.4, 102.0)
- added C4: 100n, Capacitors_SMD:C_0603_HandSoldering, F.Cu at (149.4, 93.0)
- added C5: 100n, Capacitors_SMD:C_0603_HandSoldering, F.Cu at (144.4, 97.9)
- added C6: 100n, Capacitors_SMD:C_0603_HandSoldering, F.Cu at (144.4, 96.4)
- added J1: CONN_01X06, Pin_Headers:Pin_Header_Straight_1x06_Pitch2.54mm, F.Cu at (172.1, 86.4)
- added JP1: Jumper_NC_Small, Socket_Strips:Socket_Strip_Straight_2x01_Pitch2.54mm, F.Cu at (170.4, 120.0)
- added JP2: Jumper_NC_Small, Socket_Strips:Socket_Strip_Straight_2x01_Pitch2.54mm, F.Cu at (173.5, 120.0)
- added P10: CONTROL, Connectors:USB_Micro-B, F.Cu at (176.8, 109.6)
- added P9: FX2LA, Socket_Strips:Socket_Strip_Angled_2x05_Pitch2.54mm, F.Cu at (117.3, 105.4)
- added R1: 4k7, Resistors_SMD:R_0603_HandSoldering, F.Cu at (169.3, 114.8)
- added R2: 4k7, Resistors_SMD:R_0603_HandSoldering, F.Cu at (169.3, 113.3)
- added U1: STM32L151C6TxA, Housings_QFP:TQFP-48_7x7mm_Pitch0.5mm, F.Cu at (152.8, 100.7)
- added U2: MIC550x-3.3YM5, TO_SOT_Packages_SMD:SOT-23-5_HandSoldering, F.Cu at (169.5, 109.7)
Connections:
- P1 pad 1: Net-(P1-Pad1) -> (no net)
- P1 pad 2: /IOREF -> (no net)
- P1 pad 3: /Reset -> (no net)
- P1 pad 8: /Vin -> (no net)
- P2 pad 1: /A0 -> /DAC1_OUT
- P2 pad 2: /A1 -> /DAC2_OUT
- P2 pad 3: /A2 -> /ADC_IN1
- P2 pad 4: /A3 -> (no net)
- P2 pad 5: /A4(SDA) -> /I2C_SDA
- P2 pad 6: /A5(SCL) -> /I2C_SCL
- P3 pad 1: /A5(SCL) -> (no net)
- P3 pad 10: /8 -> /I2C_SCL
- P3 pad 2: /A4(SDA) -> (no net)
- P3 pad 3: /AREF -> /SPI_CS
- P3 pad 4: GND -> /SPI_MOSI
- P3 pad 5: /13(SCK) -> /SPI_MISO
- P3 pad 6: /12(MISO) -> /SPI_SCK
- P3 pad 7: /11(**/MOSI) -> GND
- P3 pad 8: /10(**/SS) -> (no net)
- P3 pad 9: /9(**) -> /I2C_SDA
- P4 pad 1: /7 -> /UART_TX_OUT
- P4 pad 2: /6(**) -> /UART_RX_OUT
- P4 pad 3: /5(**) -> (no net)
- P4 pad 4: /4 -> (no net)
- P4 pad 5: /3(**) -> (no net)
- P4 pad 6: /2 -> (no net)
- P4 pad 7: /1(Tx) -> (no net)
- P4 pad 8: /0(Rx) -> (no net)
- P5 pad 1: Net-(P5-Pad1) -> (no net)
- P6 pad 1: Net-(P6-Pad1) -> (no net)
- P7 pad 1: Net-(P7-Pad1) -> (no net)
- P8 pad 1: Net-(P8-Pad1) -> (no net)
