File: hw1/hw1.sch (KiCad schematic (older format))
At the start: 16 parts, among them P1 Power, P10 CONTROL, P2 Analog, P3 Digital, P4 Digital, P5 CONN_01X01, P6 CONN_01X01, P7 CONN_01X01, P8 CONN_01X01, P9 FX2LA, U1 STM32L151C6TxA

Commit message: hw1: schematic "finished" ?
have I committed enough files for others to even open this?
Parts:
- added C6: 100n, Capacitors_SMD:C_0603_HandSoldering, symbol C
- added J1: CONN_01X06, Pin_Headers:Pin_Header_Straight_1x06_Pitch2.54mm, symbol CONN_01X06
- added JP1, JP2: Jumper_NC_Small, Socket_Strips:Socket_Strip_Straight_2x01_Pitch2.54mm, symbol Jumper_NC_Small
- added R1, R2: 4k7, Resistors_SMD:R_0603_HandSoldering, symbol R
- added U2: MIC550x-3.3YM5, TO_SOT_Packages_SMD:SOT-23-5_HandSoldering, symbol MIC550x-3.3YM5
- P9: footprint Connectors:IDC_Header_Straight_10pins -> Socket_Strips:Socket_Strip_Angled_2x05_Pitch2.54mm
- U1: footprint LQFP48 -> Housings_QFP:TQFP-48_7x7mm_Pitch0.5mm
Connections:
- net labels added: DAC1_OUT, DAC2_OUT, RESET_OUT, UART_RX_OUT, UART_TX_OUT, VBUS
- net labels removed: DAC1, DAC2, Reset, SPI_CSK, UART_RX, UART_TX
- wire segments 86 -> 108
- no-connect marks 12 -> 33
Other:
- note added: "Designed for a cheap FX2LA\nto be just "plugged in" for sigrok"
- note added: "Don't place this\nI dont' think we need it"
- note added: "IN/OUT from perspective of HOST\nDUT Nucleo is TARGET"
- note added: "IN/OUT is from the perspective of HOST\nDUT Nucleo is TARGET"
- note added: "STLink compatible debug"
- note added: "TODO\n[ ] Route all spare pins to _something_?"
- note added: "We're using debugger only here"
- note added: "[x] debug via via 6pin\n[ ] debug via 10x5x1.27mm cortex SMD\n"
- note removed: "TBD: debug via via 6pin/10x1.27/20x2.54? (leaning toward 6pin _and_ 10x127 smd)"
- note removed: "TODO: VBUS to 3v3 plz!"

Commit message: hw1: add in/out caps to 3v3
Parts:
- added C? (x2): 1u, Capacitors_SMD:C_0603_HandSoldering, symbol C
Connections:
- net +3V3: now also C?.1
- net +5V: now also C?.1
- net GND: now also C?.2, C?.2
Changed lines of the file:
@@
 	9400 2000 8600 2000
 Wire Wire Line
-	8850 2100 9400 2100
+	8850 2100 9300 2100
+Wire Wire Line
+	9300 2100 9400 2100
 Connection ~ 9300 2100
 Wire Wire Line
@@
 	4500 2450 4500 2350
 Wire Wire Line
-	4350 2450 4650 2450
+	4350 2450 4450 2450
+Wire Wire Line
+	4450 2450 4500 2450
+Wire Wire Line
+	4500 2450 4550 2450
+Wire Wire Line
+	4550 2450 4650 2450
 Wire Wire Line
 	4350 2450 4350 2550
@@
 	4350 6150 4350 6250
 Wire Wire Line
-	4350 6250 4650 6250
-Wire Wire Line
-	4450 6150 4450 6300
+	4350 6250 4450 6250
+Wire Wire Line
+	4450 6250 4550 6250
+Wire Wire Line
+	4550 6250 4650 6250
+Wire Wire Line
+	4450 6150 4450 6250
+Wire Wire Line
+	4450 6250 4450 6300
 Connection ~ 4450 6250
 Wire Wire Line
@@
 	2050 6850 2050 6650
 Wire Wire Line
-	1500 6850 2600 6850
+	1500 6850 1850 6850
+Wire Wire Line
+	1850 6850 2050 6850
+Wire Wire Line
+	2050 6850 2250 6850
+Wire Wire Line
+	2250 6850 2600 6850
 Connection ~ 1850 6850
 Connection ~ 2050 6850
 Connection ~ 2250 6850
 Wire Wire Line
-	1500 7150 2600 7150
+	1500 7150 1850 7150
+Wire Wire Line
+	1850 7150 2050 7150
+Wire Wire Line
+	2050 7150 2250 7150
+Wire Wire Line
+	2250 7150 2600 7150
 Connection ~ 2250 7150
 Connection ~ 1850 7150
@@
 L +3V3 #PWR014
 U 1 1 59F7B6BD
-P 6150 6800
-F 0 "#PWR014" H 6150 6650 50  0001 C CNN
-F 1 "+3V3" H 6150 6940 50  0000 C CNN
-F 2 "" H 6150 6800 50  0000 C CNN
-F 3 "" H 6150 6800 50  0000 C CNN
-	1    6150 6800
+P 6150 7000
+F 0 "#PWR014" H 6150 6850 50  0001 C CNN
+F 1 "+3V3" H 6150 7140 50  0000 C CNN
+F 2 "" H 6150 7000 50  0000 C CNN
+F 3 "" H 6150 7000 50  0000 C CNN
+	1    6150 7000
 	1    0    0    -1
 $EndComp
@@
 L GND #PWR015
 U 1 1 59F7B70C
-P 5400 7500
-F 0 "#PWR015" H 5400 7250 50  0001 C CNN
-F 1 "GND" H 5400 7350 50  0000 C CNN
-F 2 "" H 5400 7500 50  0000 C CNN
-F 3 "" H 5400 7500 50  0000 C CNN
-	1    5400 7500
-	1    0    0    -1
-$EndComp
-Wire Wire Line
-	5800 7000 6150 7000
-Wire Wire Line
-	6150 7000 6150 6800
-Wire Wire Line
-	4850 7000 5000 7000
+P 5400 7550
+F 0 "#PWR015" H 5400 7300 50  0001 C CNN
+F 1 "GND" H 5400 7400 50  0000 C CNN
+F 2 "" H 5400 7550 50  0000 C CNN
+F 3 "" H 5400 7550 50  0000 C CNN
+	1    5400 7550
+	1    0    0    -1
+$EndComp
+Wire Wire Line
+	5800 7000 6100 7000
+Wire Wire Line
+	6100 7000 6100 7000
+Wire Wire Line
+	6100 7000 6150 7000
+Wire Wire Line
+	4850 7000 4900 7000
+Wire Wire Line
+	4900 7000 5000 7000
 Wire Wire Line
 	3150 1600 3450 1600
@@
 Wire Wire Line
 	3150 1600 3150 1550
-Text Label 4900 7000 0    60   ~ 0
-VBUS
 Wire Wire Line
 	5400 7400 5400 7500
+Wire Wire Line
+	5400 7500 5400 7550
 $Comp
 L +5V #PWR016
@@
 	1    0    0    -1
 $EndComp
-Text Label 3150 1550 0    60   ~ 0
-VBUS
 $Comp
 L +5V #PWR017
@@
 Text Notes 9000 3300 0    60   ~ 0
 TODO\n[ ] Route all spare pins to _something_?
+$Comp
+L C C?
+U 1 1 5A0FC660
+P 6100 7350
+F 0 "C?" H 6125 7450 50  0000 L CNN
+F 1 "1u" H 6125 7250 50  0000 L CNN
+F 2 "Capacitors_SMD:C_0603_HandSoldering" H 6138 7200 50  0000 C CNN
+F 3 "" H 6100 7350 50  0000 C CNN
+	1    6100 7350
+	1    0    0    -1
+$EndComp
+$Comp
+L C C?
+U 1 1 5A0FC76D
+P 4900 7350
+F 0 "C?" H 4925 7450 50  0000 L CNN
+F 1 "1u" H 4925 7250 50  0000 L CNN
+F 2 "Capacitors_SMD:C_0603_HandSoldering" H 4938 7200 50  0000 C CNN
+F 3 "" H 4900 7350 50  0000 C CNN
+	1    4900 7350
+	1    0    0    -1
+$EndComp
+Wire Wire Line
+	4900 7500 5400 7500
+Wire Wire Line
+	5400 7500 6100 7500
+Connection ~ 5400 7500
+Wire Wire Line
+	6100 7200 6100 7000
+Connection ~ 6100 7000
 $EndSCHEMATC

Commit message: hw1: apparently _actually_ save the file
Parts:
- gave numbers to parts that had none: 2
Changed lines of the file:
@@
 	9400 2000 8600 2000
 Wire Wire Line
-	8850 2100 9300 2100
-Wire Wire Line
-	9300 2100 9400 2100
+	8850 2100 9400 2100
 Connection ~ 9300 2100
 Wire Wire Line
@@
 	4500 2450 4500 2350
 Wire Wire Line
-	4350 2450 4450 2450
-Wire Wire Line
-	4450 2450 4500 2450
-Wire Wire Line
-	4500 2450 4550 2450
-Wire Wire Line
-	4550 2450 4650 2450
+	4350 2450 4650 2450
 Wire Wire Line
 	4350 2450 4350 2550
@@
 	4350 6150 4350 6250
 Wire Wire Line
-	4350 6250 4450 6250
-Wire Wire Line
-	4450 6250 4550 6250
-Wire Wire Line
-	4550 6250 4650 6250
-Wire Wire Line
-	4450 6150 4450 6250
-Wire Wire Line
-	4450 6250 4450 6300
+	4350 6250 4650 6250
+Wire Wire Line
+	4450 6150 4450 6300
 Connection ~ 4450 6250
 Wire Wire Line
@@
 	2050 6850 2050 6650
 Wire Wire Line
-	1500 6850 1850 6850
-Wire Wire Line
-	1850 6850 2050 6850
-Wire Wire Line
-	2050 6850 2250 6850
-Wire Wire Line
-	2250 6850 2600 6850
+	1500 6850 2600 6850
 Connection ~ 1850 6850
 Connection ~ 2050 6850
 Connection ~ 2250 6850
 Wire Wire Line
-	1500 7150 1850 7150
-Wire Wire Line
-	1850 7150 2050 7150
-Wire Wire Line
-	2050 7150 2250 7150
-Wire Wire Line
-	2250 7150 2600 7150
+	1500 7150 2600 7150
 Connection ~ 2250 7150
 Connection ~ 1850 7150
@@
 $EndComp
 Wire Wire Line
-	5800 7000 6100 7000
-Wire Wire Line
-	6100 7000 6100 7000
-Wire Wire Line
-	6100 7000 6150 7000
-Wire Wire Line
-	4850 7000 4900 7000
-Wire Wire Line
-	4900 7000 5000 7000
+	5800 7000 6150 7000
+Wire Wire Line
+	4850 7000 5000 7000
 Wire Wire Line
 	3150 1600 3450 1600
@@
 	3150 1600 3150 1550
 Wire Wire Line
-	5400 7400 5400 7500
-Wire Wire Line
-	5400 7500 5400 7550
+	5400 7400 5400 7550
 $Comp
 L +5V #PWR016
@@
 TODO\n[ ] Route all spare pins to _something_?
 $Comp
-L C C?
+L C C8
 U 1 1 5A0FC660
 P 6100 7350
-F 0 "C?" H 6125 7450 50  0000 L CNN
+F 0 "C8" H 6125 7450 50  0000 L CNN
 F 1 "1u" H 6125 7250 50  0000 L CNN
 F 2 "Capacitors_SMD:C_0603_HandSoldering" H 6138 7200 50  0000 C CNN
@@
 $EndComp
 $Comp
-L C C?
+L C C7
 U 1 1 5A0FC76D
 P 4900 7350
-F 0 "C?" H 4925 7450 50  0000 L CNN
+F 0 "C7" H 4925 7450 50  0000 L CNN
 F 1 "1u" H 4925 7250 50  0000 L CNN
 F 2 "Capacitors_SMD:C_0603_HandSoldering" H 4938 7200 50  0000 C CNN
@@
 $EndComp
 Wire Wire Line
-	4900 7500 5400 7500
-Wire Wire Line
-	5400 7500 6100 7500
+	4900 7500 6100 7500
 Connection ~ 5400 7500
 Wire Wire Line

Commit message: hw1: begin routing.
Spun the host, laid most signal tracks.
todo: vcc, ground pour, then shuffle all LA connectors for ease of
routing.
Connections:
- net +3V3: now also R1.1, R2.1
- net VLCD: now reaches C6.1, U1.1 (VLCD)
Changed lines of the file:
@@
 $EndComp
 Wire Wire Line
-	9650 3900 9650 3800
+	9650 3800 9650 3900
 Wire Wire Line
-	9650 3800 9350 3800
+	9350 3800 9650 3800
 Wire Wire Line
 	9350 3800 9350 3900
@@
 $EndComp
 Wire Wire Line
-	700  3650 800  3650
-Wire Wire Line
-	800  3650 800  3350
-Wire Wire Line
-	800  3350 950  3350
-Wire Wire Line
 	700  3950 700  4000
 Text Notes -500 3850 0    60   ~ 0
@@
 	6100 7200 6100 7000
 Connection ~ 6100 7000
+Connection ~ 9500 3800
+Wire Wire Line
+	950  3350 700  3350
+Wire Wire Line
+	700  3350 700  3650
+Text Label 950  3350 2    60   ~ 0
+VLCD
 $EndSCHEMATC

Commit message: hw1: add crystal, more commentary
probably need a crystal for usb :)

still needs footrints, will probably be any old 3225 part.
Parts:
- added C? (x2): 18pf, Capacitors_SMD:C_0603_HandSoldering, symbol C
- added Y?: Crystal_GND24_Small, symbol Crystal_GND24_Small
Connections:
- net +3V3: no longer C2.1, C3.1, C4.1, C5.1
- net GND: now also C?.2, C?.2
- net at U1.5 (PH0/RCC_OSC_IN): now also C?.1, Y?.1
- net at U1.6 (PH1/RCC_OSC_OUT): now also C?.1, Y?.3
- new net: C2.1, C3.1, C4.1, C5.1
- no-connect marks 33 -> 31
Other:
- note added: "L1/F303/L4 in qfp48 are all compatible with this layout\n(but f3 needs external pullup on USB-DP)"
- note added: "Not needed on L1, but needed for L4/F3"
- note removed: "Don't place this\nI dont' think we need it"

Commit message: hw1: continued, just intermediate progress save
wtf kicad, why aren't my grounds connected?!
Parts:
- Y1: renamed from Y?; footprint (none) -> Crystals:Crystal_SMD_SeikoEpson_FA238-4pin_3.2x2.5mm
- gave numbers to parts that had none: 2
Connections:
- net +3V3: now also C2.1, C3.1, C4.1, C5.1
- net I2C_SCL: now also P9.2 (P2); no longer P9.1 (P1)
- net I2C_SDA: now also P9.1 (P1); no longer P9.2 (P2)
- net SPI_CS: now also P9.8 (P8); no longer P9.6 (P6)
- net SPI_MISO: now also P9.6 (P6); no longer P9.4 (P4)
- net SPI_SCK: now also P9.7 (P7); no longer P9.3 (P3)
- net UART_RX_OUT: now also P9.4 (P4); no longer P9.7 (P7)
- net UART_TX_OUT: now also P9.3 (P3); no longer P9.8 (P8)
- net at C9.1, U1.5 (PH0/RCC_OSC_IN): now also Y1.3; no longer Y1.1
- net at C10.1, U1.6 (PH1/RCC_OSC_OUT): now also Y1.1; no longer Y1.3
Changed lines of the file:
@@
 	1250 1350 1200 1350
 Text Label 1200 1050 2    60   ~ 0
+I2C_SDA
+Text Label 1800 1050 0    60   ~ 0
 I2C_SCL
-Text Label 1800 1050 0    60   ~ 0
-I2C_SDA
 Text Label 1200 1150 2    60   ~ 0
-SPI_SCK
+UART_TX_OUT
 Text Label 1200 1250 2    60   ~ 0
 SPI_MOSI
 Text Label 1800 1150 0    60   ~ 0
+UART_RX_OUT
+Text Label 1800 1250 0    60   ~ 0
 SPI_MISO
-Text Label 1800 1250 0    60   ~ 0
-SPI_CS
 Text Label 1200 1350 2    60   ~ 0
-UART_RX_OUT
+SPI_SCK
 Text Notes 500  2100 0    60   Italic 0
 NOTE: this can be freely routed to do whatever's possible!\nPotentially:\nJumpers to select what you're connecting here?\n(but non-ideal)
@@
 L +3V3 #PWR010
 U 1 1 58CF46D6
-P 2450 6800
-F 0 "#PWR010" H 2450 6650 50  0001 C CNN
-F 1 "+3V3" H 2450 6940 50  0000 C CNN
-F 2 "" H 2450 6800 50  0000 C CNN
-F 3 "" H 2450 6800 50  0000 C CNN
-	1    2450 6800
+P 2050 6650
+F 0 "#PWR010" H 2050 6500 50  0001 C CNN
+F 1 "+3V3" H 2050 6790 50  0000 C CNN
+F 2 "" H 2050 6650 50  0000 C CNN
+F 3 "" H 2050 6650 50  0000 C CNN
+	1    2050 6650
 	1    0    0    -1
 $EndComp
@@
 IN/OUT is from the perspective of HOST\nDUT Nucleo is TARGET
 Text Label 1800 1350 0    60   ~ 0
-UART_TX_OUT
+SPI_CS
 Text Label 5600 1250 0    60   ~ 0
 SWCLK
@@
 L1/F303/L4 in qfp48 are all compatible with this layout\n(but f3 needs external pullup on USB-DP)
 $Comp
-L Crystal_GND24_Small Y?
+L Crystal_GND24_Small Y1
 U 1 1 5A137095
 P 800 3800
-F 0 "Y?" H 850 3975 50  0000 L CNN
+F 0 "Y1" H 850 3975 50  0000 L CNN
 F 1 "Crystal_GND24_Small" H 850 3900 50  0000 L CNN
-F 2 "" H 800 3800 50  0001 C CNN
+F 2 "Crystals:Crystal_SMD_SeikoEpson_FA238-4pin_3.2x2.5mm" H 800 3800 50  0001 C CNN
 F 3 "" H 800 3800 50  0001 C CNN
 	1    800  3800
-	0    1    1    0
+	0    -1   -1   0
 $EndComp
 Wire Wire Line
@@
 	1350 3800 1150 3800
 Wire Wire Line
-	1150 3900 1150 3800
-Wire Wire Line
-	750  3900 1150 3900
-$Comp
-L C C?
+	1150 3800 1150 3900
+Wire Wire Line
+	1150 3900 750  3900
+$Comp
+L C C10
 U 1 1 5A1373B8
 P 750 4150
-F 0 "C?" H 775 4250 50  0000 L CNN
+F 0 "C10" H 775 4250 50  0000 L CNN
 F 1 "18pf" H 775 4050 50  0000 L CNN
 F 2 "Capacitors_SMD:C_0603_HandSoldering" H 788 4000 50  0000 C CNN
@@
 $EndComp
 $Comp
-L C C?
+L C C9
 U 1 1 5A137455
 P 550 4150
-F 0 "C?" H 575 4250 50  0000 L CNN
+F 0 "C9" H 575 4250 50  0000 L CNN
 F 1 "18pf" H 575 4050 50  0000 L CNN
 F 2 "Capacitors_SMD:C_0603_HandSoldering" H 588 4000 50  0000 C CNN
@@
 $EndComp
 $Comp
-L GND #PWR?
+L GND #PWR022
 U 1 1 5A137592
 P 650 4400
-F 0 "#PWR?" H 650 4150 50  0001 C CNN
+F 0 "#PWR022" H 650 4150 50  0001 C CNN
 F 1 "GND" H 650 4250 50  0000 C CNN
 F 2 "" H 650 4400 50  0000 C CNN
@@
 Connection ~ 650  4300
 Wire Wire Line
-	750  4000 750  3900
+	750  3900 750  4000
 Connection ~ 800  3900
 $EndSCHEMATC

Commit message: "fix" grounds by tracks into pour
"finish" routing, ignore DRC violations from disconnected usb shield on
pin 6.

Add boot0 jumper pad "just in case" but really kinda dumb, we've got a
debug header on it. Why bother with this?

Change paper size in schema to get more space.

TODO: add silk?
TODO: replace "arduino" shape with just the pinpoints.
Parts:
- added J2: CONN_01X01_MALE, Wire_Pads:SolderWirePad_single_0-8mmDrill, symbol CONN_01X01_MALE
- added J3: CONN_01X02, Pin_Headers:Pin_Header_Straight_1x02_Pitch2.54mm, symbol CONN_01X02
- added JP3: Jumper_NC_Small, Socket_Strips:Socket_Strip_Straight_2x01_Pitch2.54mm, symbol Jumper_NC_Small
Connections:
- wire segments 116 -> 114
- no-connect marks 31 -> 33
Other:
- note added: "5V"
- note added: "D15 (_ALSO_ SCL)\nD14 (_ALSO_ SDA)"
- note added: "ONLY GROUND BETWEEN BOARDS by default!\nIntended for both to have their own USB\nOption for debug only, with power FROM target"
- note added: "Probe points, for\nbus tracing USB"
- note added: "We're using debugger only here\n(but be safe)"
- note removed: "D15 (SCL)\nD14 (SDA)"
- note removed: "ONLY GROUND BETWEEN BOARDS\nBoth will be powered by their own USB.\n(We're not interested in bootloading the target....\nyet...?)"
- note removed: "We're using debugger only here"

Commit message: hw1: test points, cleanup 3d view
Fixed boot0 to be tied down, will be programmed via swd.
Added test points for spare pins where easy
Fixed some footprints to make the 3d view pretty.
Parts:
- removed J2: CONN_01X01_MALE, Wire_Pads:SolderWirePad_single_0-8mmDrill, symbol CONN_01X01_MALE
- added J10, J11, J2, J3, J4, J5, J7, J8, J9: TEST_1P, Measurement_Points:Measurement_Point_Round-TH_Small, symbol TEST_1P
- JP1, JP2, JP3: footprint Socket_Strips:Socket_Strip_Straight_2x01_Pitch2.54mm -> Pin_Headers:Pin_Header_Straight_1x02_Pitch2.54mm
- P11: renamed from J1; footprint Pin_Headers:Pin_Header_Straight_1x06_Pitch2.54mm -> Socket_Strips:Socket_Strip_Straight_1x06_Pitch2.54mm
- renumbered J3 to J1
Connections:
- wire segments 114 -> 123
- no-connect marks 33 -> 23
Other:
- note added: "Bootloader wut?"
- note added: "no need for rtc\nthis is the host board"
- note removed: "We're using debugger only here\n(but be safe)"
Changed lines of the file:
@@
 Wire Wire Line
 	1050 4400 900  4400
-NoConn ~ 2550 5700
-NoConn ~ 2550 5800
 NoConn ~ 2550 5500
 NoConn ~ 2550 5400
@@
 Connection ~ 7700 9950
 $Comp
-L CONN_01X06 J1
+L CONN_01X06 P11
 U 1 1 59F7E088
 P 6850 1300
-F 0 "J1" H 6850 1650 50  0000 C CNN
+F 0 "P11" H 6850 1650 50  0000 C CNN
 F 1 "CONN_01X06" V 6950 1300 50  0000 C CNN
-F 2 "Pin_Headers:Pin_Header_Straight_1x06_Pitch2.54mm" H 6850 1300 50  0001 C CNN
+F 2 "Socket_Strips:Socket_Strip_Straight_1x06_Pitch2.54mm" H 6850 1300 50  0001 C CNN
 F 3 "" H 6850 1300 50  0001 C CNN
 	1    6850 1300
@@
 Text Notes 6700 850  0    60   ~ 0
 STLink compatible debug
-NoConn ~ 9750 5700
-NoConn ~ 9750 5800
-NoConn ~ 9750 6500
-NoConn ~ 9750 6600
-NoConn ~ 9750 6700
 NoConn ~ 9750 7200
-NoConn ~ 2550 6800
-NoConn ~ 2550 6700
 NoConn ~ 2550 6400
 NoConn ~ 2550 6300
@@
 F 0 "JP1" H 10600 10130 50  0000 C CNN
 F 1 "Jumper_NC_Small" H 10610 9990 50  0000 C CNN
-F 2 "Socket_Strips:Socket_Strip_Straight_2x01_Pitch2.54mm" H 10600 10050 50  0001 C CNN
+F 2 "Pin_Headers:Pin_Header_Straight_1x02_Pitch2.54mm" H 10600 10050 50  0001 C CNN
 F 3 "" H 10600 10050 50  0001 C CNN
 	1    10600 10050
@@
 F 0 "JP2" H 10900 10130 50  0000 C CNN
 F 1 "Jumper_NC_Small" H 10910 9990 50  0000 C CNN
-F 2 "Socket_Strips:Socket_Strip_Straight_2x01_Pitch2.54mm" H 10900 10050 50  0001 C CNN
+F 2 "Pin_Headers:Pin_Header_Straight_1x02_Pitch2.54mm" H 10900 10050 50  0001 C CNN
 F 3 "" H 10900 10050 50  0001 C CNN
 	1    10900 10050
@@
 	12500 2400 12400 2400
 NoConn ~ 12400 2400
-NoConn ~ 2550 5900
 Text Notes 2950 4600 0    39   ~ 0
-We're using debugger only here\n(but be safe)
+Bootloader wut?
 $Comp
 L C C6
@@
 F 0 "JP3" H 12050 2080 50  0000 C CNN
 F 1 "Jumper_NC_Small" H 12060 1940 50  0000 C CNN
-F 2 "Socket_Strips:Socket_Strip_Straight_2x01_Pitch2.54mm" H 12050 2000 50  0001 C CNN
+F 2 "Pin_Headers:Pin_Header_Straight_1x02_Pitch2.54mm" H 12050 2000 50  0001 C CNN
 F 3 "" H 12050 2000 50  0001 C CNN
 	1    12050 2000
@@
 	11800 2000 11800 1550
 $Comp
-L CONN_01X02 J3
+L CONN_01X02 J1
 U 1 1 5A36EBE0
 P 4850 2350
-F 0 "J3" H 4850 2500 50  0000 C CNN
+F 0 "J1" H 4850 2500 50  0000 C CNN
 F 1 "CONN_01X02" V 4950 2350 50  0000 C CNN
 F 2 "Pin_Headers:Pin_Header_Straight_1x02_Pitch2.54mm" H 4850 2350 50  0001 C CNN
@@
 Text Notes 4550 2700 0    60   ~ 0
 Probe points, for\nbus tracing USB
-$Comp
-L CONN_01X01_MALE J2
-U 1 1 5A36F13B
-P 2150 4600
-F 0 "J2" H 2150 4675 50  0000 C CNN
-F 1 "CONN_01X01_MALE" H 2150 4500 50  0000 C CNN
-F 2 "Wire_Pads:SolderWirePad_single_0-8mmDrill" H 2150 4600 50  0001 C CNN
-F 3 "" H 2150 4600 50  0001 C CNN
-	1    2150 4600
-	1    0    0    -1
-$EndComp
-Wire Wire Line
-	2550 4600 2450 4600
+Wire Wire Line
+	2550 4600 2200 4600
 Wire Wire Line
 	1450 4900 1450 5300
@@
 NoConn ~ 13300 1300
 NoConn ~ 13300 1400
+$Comp
+L GND #PWR022
+U 1 1 5A43A55C
+P 2200 4600
+F 0 "#PWR022" H 2200 4350 50  0001 C CNN
+F 1 "GND" H 2200 4450 50  0000 C CNN
+F 2 "" H 2200 4600 50  0000 C CNN
+F 3 "" H 2200 4600 50  0000 C CNN
+	1    2200 4600
+	1    0    0    -1
+$EndComp
+$Comp
+L TEST_1P J2
+U 1 1 5A43D04F
+P 2500 5700
+F 0 "J2" H 2500 5970 50  0000 C CNN
+F 1 "TEST_1P" H 2500 5900 50  0000 C CNN
+F 2 "Measurement_Points:Measurement_Point_Round-TH_Small" H 2700 5700 50  0001 C CNN
+F 3 "" H 2700 5700 50  0001 C CNN
+	1    2500 5700
+	0    -1   -1   0
+$EndComp
+$Comp
+L TEST_1P J3
+U 1 1 5A43D328
+P 2300 5800
+F 0 "J3" H 2300 6070 50  0000 C CNN
+F 1 "TEST_1P" H 2300 6000 50  0000 C CNN
+F 2 "Measurement_Points:Measurement_Point_Round-TH_Small" H 2500 5800 50  0001 C CNN
+F 3 "" H 2500 5800 50  0001 C CNN
+	1    2300 5800
+	0    -1   -1   0
+$EndComp
+$Comp
+L TEST_1P J4
+U 1 1 5A43D40B
+P 2250 6700
+F 0 "J4" H 2250 6970 50  0000 C CNN
+F 1 "TEST_1P" H 2250 6900 50  0000 C CNN
+F 2 "Measurement_Points:Measurement_Point_Round-TH_Small" H 2450 6700 50  0001 C CNN
+F 3 "" H 2450 6700 50  0001 C CNN
+	1    2250 6700
+	0    -1   -1   0
+$EndComp
+$Comp
+L TEST_1P J5
+U 1 1 5A43D49D
+P 2100 6800
+F 0 "J5" H 2100 7070 50  0000 C CNN
+F 1 "TEST_1P" H 2100 7000 50  0000 C CNN
+F 2 "Measurement_Points:Measurement_Point_Round-TH_Small" H 2300 6800 50  0001 C CNN
+F 3 "" H 2300 6800 50  0001 C CNN
+	1    2100 6800
+	0    -1   -1   0
+$EndComp
+Wire Wire Line
+	2500 5700 2550 5700
+Wire Wire Line
+	2550 5800 2300 5800
+Wire Wire Line
+	2550 6700 2250 6700
+Wire Wire Line
+	2550 6800 2100 6800
+$Comp
+L TEST_1P J7
+U 1 1 5A43EE7B
+P 10100 6500
+F 0 "J7" H 10100 6770 50  0000 C CNN
+F 1 "TEST_1P" H 10100 6700 50  0000 C CNN
+F 2 "Measurement_Points:Measurement_Point_Round-TH_Small" H 10300 6500 50  0001 C CNN
+F 3 "" H 10300 6500 50  0001 C CNN
+	1    10100 6500
+	0    1    1    0
+$EndComp
+$Comp
+L TEST_1P J8
+U 1 1 5A43F060
+P 10250 6600
+F 0 "J8" H 10250 6870 50  0000 C CNN
+F 1 "TEST_1P" H 10250 6800 50  0000 C CNN
+F 2 "Measurement_Points:Measurement_Point_Round-TH_Small" H 10450 6600 50  0001 C CNN
+F 3 "" H 10450 6600 50  0001 C CNN
+	1    10250 6600
+	0    1    1    0
+$EndComp
+$Comp
+L TEST_1P J9
+U 1 1 5A43F0E2
+P 10400 6700
+F 0 "J9" H 10400 6970 50  0000 C CNN
+F 1 "TEST_1P" H 10400 6900 50  0000 C CNN
+F 2 "Measurement_Points:Measurement_Point_Round-TH_Small" H 10600 6700 50  0001 C CNN
+F 3 "" H 10600 6700 50  0001 C CNN
+	1    10400 6700
+	0    1    1    0
+$EndComp
+Wire Wire Line
+	9750 6500 10100 6500
+Wire Wire Line
+	9750 6600 10250 6600
+Wire Wire Line
+	9750 6700 10400 6700
+$Comp
+L TEST_1P J10
+U 1 1 5A43FB1F
+P 10300 5700
+F 0 "J10" H 10300 5970 50  0000 C CNN
+F 1 "TEST_1P" H 10300 5900 50  0000 C CNN
+F 2 "Measurement_Points:Measurement_Point_Round-TH_Small" H 10500 5700 50  0001 C CNN
+F 3 "" H 10500 5700 50  0001 C CNN
+	1    10300 5700
+	0    1    1    0
+$EndComp
+$Comp
+L TEST_1P J11
+U 1 1 5A43FBC5
+P 10500 5800
+F 0 "J11" H 10500 6070 50  0000 C CNN
+F 1 "TEST_1P" H 10500 6000 50  0000 C CNN
+F 2 "Measurement_Points:Measurement_Point_Round-TH_Small" H 10700 5800 50  0001 C CNN
+F 3 "" H 10700 5800 50  0001 C CNN
+	1    10500 5800
+	0    1    1    0
+$EndComp
+Wire Wire Line
+	9750 5700 10300 5700
+Wire Wire Line
+	9750 5800 10500 5800
+Text Notes 5900 5400 0    60   ~ 0
+no need for rtc\nthis is the host board
 $EndSCHEMATC
