File: hw1/hw1.sch (KiCad schematic (older format))
At the start: 39 parts, among them J1 CONN_01X02, J10 TEST_1P, J11 TEST_1P, J2 TEST_1P, J3 TEST_1P, J4 TEST_1P, J5 TEST_1P, J7 TEST_1P, J8 TEST_1P, J9 TEST_1P, P1 Power, P10 CONTROL, P11 CONN_01X06, P2 Analog, P3 Digital, P4 Digital, P5 CONN_01X01, P6 CONN_01X01, P7 CONN_01X01, P8 CONN_01X01, P9 FX2LA, U1 STM32L151C6TxA, U2 MIC550x-3.3YM5, Y1 Crystal_GND24_Small

Commit message: hw1: drop arduinno style holes and board shape
More to go, nno need for the silk and dead shapes, we just needed the
pin spacings
Parts:
- removed P5, P6, P7, P8: CONN_01X01, Socket_Arduino_Uno:Arduino_1pin, symbol CONN_01X01
Connections:
- no-connect marks 23 -> 20
Other:
- note removed: "Holes"
Changed lines of the file:
@@
 AREF
 NoConn ~ 12500 1700
-Text Notes 13950 1100 0    60   ~ 0
-Holes
 Text Notes 11650 850  0    60   ~ 0
 Arduino UNOr3 pins\nAs used on Nucleo64 boards\n
@@
 	1    0    0    -1
 $EndComp
-$Comp
-L CONN_01X01 P5
-U 1 1 56D71177
-P 13900 750
-F 0 "P5" V 14000 750 50  0000 C CNN
-F 1 "CONN_01X01" V 14000 750 50  0001 C CNN
-F 2 "Socket_Arduino_Uno:Arduino_1pin" H 13900 750 50  0001 C CNN
-F 3 "" H 13900 750 50  0000 C CNN
-	1    13900 750
-	0    -1   -1   0
-$EndComp
-$Comp
-L CONN_01X01 P6
-U 1 1 56D71274
-P 14000 750
-F 0 "P6" V 14100 750 50  0000 C CNN
-F 1 "CONN_01X01" V 14100 750 50  0001 C CNN
-F 2 "Socket_Arduino_Uno:Arduino_1pin" H 14000 750 50  0001 C CNN
-F 3 "" H 14000 750 50  0000 C CNN
-	1    14000 750
-	0    -1   -1   0
-$EndComp
-$Comp
-L CONN_01X01 P7
-U 1 1 56D712A8
-P 14100 750
-F 0 "P7" V 14200 750 50  0000 C CNN
-F 1 "CONN_01X01" V 14200 750 50  0001 C CNN
-F 2 "Socket_Arduino_Uno:Arduino_1pin" H 14100 750 50  0001 C CNN
-F 3 "" H 14100 750 50  0000 C CNN
-	1    14100 750
-	0    -1   -1   0
-$EndComp
-$Comp
-L CONN_01X01 P8
-U 1 1 56D712DB
-P 14200 750
-F 0 "P8" V 14300 750 50  0000 C CNN
-F 1 "CONN_01X01" V 14300 750 50  0001 C CNN
-F 2 "Socket_Arduino_Uno:Arduino_1pin" H 14200 750 50  0001 C CNN
-F 3 "" H 14200 750 50  0000 C CNN
-	1    14200 750
-	0    -1   -1   0
-$EndComp
-NoConn ~ 13900 950
-NoConn ~ 14000 950
-NoConn ~ 14100 950
-NoConn ~ 14200 950
 $Comp
 L CONN_01X08 P4
@@
 Wire Wire Line
 	12500 1900 12400 1900
-Wire Notes Line
-	14300 1100 13800 1100
-Wire Notes Line
-	13800 1100 13800 600
 Wire Wire Line
 	6100 3900 6100 3800
@@
 Connection ~ 8900 9950
 Connection ~ 10750 9500
-Wire Wire Line
-	1350 4800 2550 4800
 Text Label 2550 4800 2    60   ~ 0
 VLCD
@@
 Text Notes 5900 5400 0    60   ~ 0
 no need for rtc\nthis is the host board
+Wire Wire Line
+	2550 4800 1350 4800
+NoConn ~ 2550 5900
 $EndSCHEMATC

Commit message: hw1: more silk cleanup
Parts:
- renumbered J10 to PA0, J11 to PA1, J9 to PA10, J7 to PA8, J8 to PA9, J2 to PB0, J3 to PB1, J4 to PB10, J5 to PB11
Other:
- note added: "TODO Jumper RTS/CTS over to I2C on fx2 port?"
Changed lines of the file:
@@
 $EndComp
 $Comp
-L TEST_1P J2
+L TEST_1P PB0
 U 1 1 5A43D04F
 P 2500 5700
-F 0 "J2" H 2500 5970 50  0000 C CNN
+F 0 "PB0" H 2500 5970 50  0000 C CNN
 F 1 "TEST_1P" H 2500 5900 50  0000 C CNN
 F 2 "Measurement_Points:Measurement_Point_Round-TH_Small" H 2700 5700 50  0001 C CNN
@@
 $EndComp
 $Comp
-L TEST_1P J3
+L TEST_1P PB1
 U 1 1 5A43D328
 P 2300 5800
-F 0 "J3" H 2300 6070 50  0000 C CNN
+F 0 "PB1" H 2300 6070 50  0000 C CNN
 F 1 "TEST_1P" H 2300 6000 50  0000 C CNN
 F 2 "Measurement_Points:Measurement_Point_Round-TH_Small" H 2500 5800 50  0001 C CNN
@@
 $EndComp
 $Comp
-L TEST_1P J4
+L TEST_1P PB10
 U 1 1 5A43D40B
 P 2250 6700
-F 0 "J4" H 2250 6970 50  0000 C CNN
+F 0 "PB10" H 2250 6970 50  0000 C CNN
 F 1 "TEST_1P" H 2250 6900 50  0000 C CNN
 F 2 "Measurement_Points:Measurement_Point_Round-TH_Small" H 2450 6700 50  0001 C CNN
@@
 $EndComp
 $Comp
-L TEST_1P J5
+L TEST_1P PB11
 U 1 1 5A43D49D
 P 2100 6800
-F 0 "J5" H 2100 7070 50  0000 C CNN
+F 0 "PB11" H 2100 7070 50  0000 C CNN
 F 1 "TEST_1P" H 2100 7000 50  0000 C CNN
 F 2 "Measurement_Points:Measurement_Point_Round-TH_Small" H 2300 6800 50  0001 C CNN
@@
 	2550 6800 2100 6800
 $Comp
-L TEST_1P J7
+L TEST_1P PA8
 U 1 1 5A43EE7B
 P 10100 6500
-F 0 "J7" H 10100 6770 50  0000 C CNN
+F 0 "PA8" H 10100 6770 50  0000 C CNN
 F 1 "TEST_1P" H 10100 6700 50  0000 C CNN
 F 2 "Measurement_Points:Measurement_Point_Round-TH_Small" H 10300 6500 50  0001 C CNN
@@
 $EndComp
 $Comp
-L TEST_1P J8
+L TEST_1P PA9
 U 1 1 5A43F060
 P 10250 6600
-F 0 "J8" H 10250 6870 50  0000 C CNN
+F 0 "PA9" H 10250 6870 50  0000 C CNN
 F 1 "TEST_1P" H 10250 6800 50  0000 C CNN
 F 2 "Measurement_Points:Measurement_Point_Round-TH_Small" H 10450 6600 50  0001 C CNN
@@
 $EndComp
 $Comp
-L TEST_1P J9
+L TEST_1P PA10
 U 1 1 5A43F0E2
 P 10400 6700
-F 0 "J9" H 10400 6970 50  0000 C CNN
+F 0 "PA10" H 10400 6970 50  0000 C CNN
 F 1 "TEST_1P" H 10400 6900 50  0000 C CNN
 F 2 "Measurement_Points:Measurement_Point_Round-TH_Small" H 10600 6700 50  0001 C CNN
@@
 	9750 6700 10400 6700
 $Comp
-L TEST_1P J10
+L TEST_1P PA0
 U 1 1 5A43FB1F
 P 10300 5700
-F 0 "J10" H 10300 5970 50  0000 C CNN
+F 0 "PA0" H 10300 5970 50  0000 C CNN
 F 1 "TEST_1P" H 10300 5900 50  0000 C CNN
 F 2 "Measurement_Points:Measurement_Point_Round-TH_Small" H 10500 5700 50  0001 C CNN
@@
 $EndComp
 $Comp
-L TEST_1P J11
+L TEST_1P PA1
 U 1 1 5A43FBC5
 P 10500 5800
-F 0 "J11" H 10500 6070 50  0000 C CNN
+F 0 "PA1" H 10500 6070 50  0000 C CNN
 F 1 "TEST_1P" H 10500 6000 50  0000 C CNN
 F 2 "Measurement_Points:Measurement_Point_Round-TH_Small" H 10700 5800 50  0001 C CNN
@@
 	2550 4800 1350 4800
 NoConn ~ 2550 5900
+Text Notes 10900 5750 0    60   ~ 0
+TODO Jumper RTS/CTS over to I2C on fx2 port?
 $EndSCHEMATC

Commit message: hw1: discover reversed numbering on arduino connectors
joy.  Fixed now against nucleo64 manuals.
Connections:
- net 2: now also P4.6 (P6); no longer P4.3 (P3)
- net 3(**): now also P4.5 (P5); no longer P4.4 (P4)
- net 4: now also P4.4 (P4); no longer P4.5 (P5)
- net 5(**): now also P4.3 (P3); no longer P4.6 (P6)
- net 6(**): now also P4.2 (P2); no longer P4.7 (P7)
- net 7: now also P4.1 (P1); no longer P4.8 (P8)
- net 8: now also P3.10 (P10); no longer P3.1 (P1)
- net 9(**): now also P3.9 (P9); no longer P3.2 (P2)
- net AREF: now also P3.3 (P3); no longer P3.8 (P8)
- net GND: now also P3.4 (P4); no longer P3.7 (P7)
- net SPI_CS: now also P3.8 (P8); no longer P3.3 (P3)
- net SPI_MISO: now also P3.6 (P6); no longer P3.5 (P5)
- net SPI_MOSI: now also P3.7 (P7); no longer P3.4 (P4)
- net SPI_SCK: now also P3.5 (P5); no longer P3.6 (P6)
- net UART_RX_OUT: now also P4.7 (P7); no longer P4.2 (P2)
- net UART_TX_OUT: now also P4.8 (P8); no longer P4.1 (P1)
Changed lines of the file:
@@
 F 3 "" H 13100 2750 50  0000 C CNN
 	1    13100 2750
-	-1   0    0    1
+	-1   0    0    -1
 $EndComp
 $Comp
@@
 F 3 "" H 13100 1750 50  0000 C CNN
 	1    13100 1750
-	-1   0    0    1
+	-1   0    0    -1
 $EndComp
 Text Notes 12800 1700 0    60   ~ 0
@@
 Wire Wire Line
 	1050 4800 900  4800
-Text Notes -50  4450 0    60   ~ 0
+Text Notes 2950 4800 0    60   ~ 0
 Not needed on L1, but needed for L4/F3
 Text Notes 12100 3400 0    60   ~ 0

Commit message: hw1: use explicit 10103594-0001LF part
better fit
Parts:
- P10: footprint Connectors:USB_Micro-B -> Connectors:USB_Micro-B_10103594-0001LF
Changed lines of the file:
@@
 F 0 "P10" H 5225 1275 50  0000 C CNN
 F 1 "CONTROL" H 4900 1600 50  0000 C CNN
-F 2 "Connectors:USB_Micro-B" V 4850 1300 50  0001 C CNN
+F 2 "Connectors:USB_Micro-B_10103594-0001LF" V 4850 1300 50  0001 C CNN
 F 3 "" V 4850 1300 50  0000 C CNN
 	1    4900 1400

Commit message: hw1: add exampe part number for fx2la part number
Parts:
- P9: female-RA (none) -> Wurth 613010243121
Changed lines of the file:
@@
 F 2 "Socket_Strips:Socket_Strip_Angled_2x05_Pitch2.54mm" H 1850 250 50  0001 C CNN
 F 3 "" H 1850 250 50  0000 C CNN
+F 4 "Wurth 613010243121" H 1850 1450 60  0001 C CNN "female-RA"
 	1    1850 1450
 	1    0    0    -1
